File: hardware/d11_usb_mini.brd (EAGLE design)
At the start: 17.4 x 12.2 mm, 20 parts, among them IC1 MIC5504-3.3, IC2 ATSAMD11C, J5 SIO, J6 SCK, J7 RST, J8 GND, X1 MINI-USB-32005-201

Commit message: Minor hardware changes + bootloader mode
Parts:
- LED1: device led:CHIPLED_0603 -> ataradov_led:SMD0603
- turned LED1 to 0 degrees
Connections:
- net +3V3: now also LED1.1; no longer LED1.A
- net N$6: now also LED1.2; no longer LED1.C
Other:
- board text added: "1/26/17"
- board text removed: "1/24/17"
Changed lines of the file:
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@@
 <wire x1="0" y1="12.182" x2="0" y2="0" width="0.1524" layer="20"/>
 <circle x="15.748" y="9.906" radius="1.143" width="0.3048" layer="27"/>
-<text x="12.7" y="0.508" size="0.762" layer="28" font="vector" rot="MR0" align="bottom-center">1/24/17</text>
+<text x="12.7" y="0.508" size="0.762" layer="28" font="vector" rot="MR0" align="bottom-center">1/26/17</text>
 <text x="4.572" y="10.16" size="1.27" layer="28" font="vector" rot="MR0" align="bottom-center">AT</text>
 </plain>
@@
 <element name="TP3" library="ataradov_misc" package="TP-1.27MM" value="" x="6.858" y="1.524" rot="MR0"/>
 <element name="TP4" library="ataradov_misc" package="TP-1.27MM" value="" x="1.778" y="1.524" rot="MR0"/>
-<element name="LED1" library="led" package="CHIPLED_0603" value="" x="11.43" y="3.302" rot="R270"/>
+<element name="LED1" library="ataradov_led" package="SMD0603" value="" x="11.43" y="3.302"/>
 </elements>
 <signals>
@@
 <wire x1="12.38" y1="4.976" x2="12.38" y2="6.574" width="0.254" layer="1"/>
 <wire x1="12.23" y1="3.302" x2="12.23" y2="4.826" width="0.254" layer="16"/>
-<wire x1="10.668" y1="3.302" x2="10.68" y2="3.302" width="0.254" layer="1"/>
-<wire x1="10.68" y1="3.302" x2="10.706" y2="3.302" width="0.254" layer="1"/>
-<wire x1="10.706" y1="3.302" x2="10.706" y2="3.01" width="0.254" layer="1"/>
-<wire x1="10.706" y1="3.01" x2="11.43" y2="2.286" width="0.254" layer="1"/>
-<wire x1="11.43" y1="2.286" x2="11.43" y2="2.032" width="0.254" layer="1"/>
 <via x="11.43" y="2.032" extent="1-16" drill="0.508" diameter="0.8636"/>
 <wire x1="11.43" y1="2.032" x2="11.43" y2="2.502" width="0.254" layer="16"/>
 <wire x1="11.43" y1="2.502" x2="12.23" y2="3.302" width="0.254" layer="16"/>
+<contactref element="LED1" pad="1"/>
+<wire x1="10.63" y1="3.302" x2="6.096" y2="3.302" width="0.254" layer="1"/>
+<wire x1="10.63" y1="3.302" x2="10.63" y2="2.832" width="0.254" layer="1"/>
+<wire x1="10.63" y1="2.832" x2="10.668" y2="2.794" width="0.254" layer="1"/>
+<wire x1="10.668" y1="2.794" x2="11.43" y2="2.032" width="0.254" layer="1"/>
 <wire x1="12.23" y1="4.826" x2="12.192" y2="4.826" width="0.254" layer="1"/>
 <wire x1="12.192" y1="4.826" x2="10.668" y2="3.302" width="0.254" layer="1"/>
-<contactref element="LED1" pad="A"/>
-<wire x1="6.096" y1="3.302" x2="10.68" y2="3.302" width="0.254" layer="1"/>
+<wire x1="10.668" y1="3.302" x2="10.668" y2="2.794" width="0.254" layer="1"/>
 </signal>
 <signal name="SWDIO">
@@
 <signal name="N$6">
 <contactref element="R7" pad="2"/>
-<contactref element="LED1" pad="C"/>
 <wire x1="12.23" y1="6.35" x2="12.954" y2="6.35" width="0.254" layer="16"/>
 <wire x1="12.954" y1="6.35" x2="13.208" y2="6.096" width="0.254" layer="16"/>
@@
 <wire x1="12.954" y1="2.032" x2="12.7" y2="2.032" width="0.254" layer="16"/>
 <via x="12.7" y="2.032" extent="1-16" drill="0.508" diameter="0.8636"/>
-<wire x1="12.7" y1="2.032" x2="12.18" y2="2.552" width="0.254" layer="1"/>
-<wire x1="12.18" y1="2.552" x2="12.18" y2="3.302" width="0.254" layer="1"/>
+<contactref element="LED1" pad="2"/>
+<wire x1="12.23" y1="3.302" x2="12.23" y2="2.502" width="0.254" layer="1"/>
+<wire x1="12.23" y1="2.502" x2="12.7" y2="2.032" width="0.254" layer="1"/>
 </signal>
 </signals>
